File: charge_amplifier/charge_amplifier.kicad_pcb (KiCad board)
At the start: 2 copper layers, 36.6 x 23.4 mm, 31 parts, among them J1 TEST_1P, J2 TEST_1P, J3 Conn_01x02, J4 Conn_01x02, J5 Conn_01x02, J6 TEST_1P, U1 TL072

Commit message: finalize layout
Parts:
- added G***: LOGO, lib_fp:LG_MARK_025in, B.Cu at (93.1, 140.3)
Routing:
- added copper zone on B.Cu, net GNDA
Other:
- rule pad_to_mask_clearance: 0.2 -> 0.0508
- board text added: "Batt"
- board text added: "Cg. Amp"
- board text added: "Charge Amplifier Leeman Geophysical LLC Rev.A - November 2017"
- board text added: "GND"
- board text added: "Out"
Changed lines of the file:
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@@
     (area 78.664999 128.956999 115.391001 152.475001)
     (thickness 1.6)
-    (drawings 5)
+    (drawings 12)
     (tracks 113)
     (zones 0)
-    (modules 31)
+    (modules 32)
     (nets 16)
   )
@@
   )
   (setup
-    (last_trace_width 0.508)
+    (last_trace_width 0.1524)
     (user_trace_width 0.1524)
     (user_trace_width 0.254)
@@
     (pad_size 3 3)
     (pad_drill 2.05)
-    (pad_to_mask_clearance 0.2)
+    (pad_to_mask_clearance 0.0508)
     (aux_axis_origin 0 0)
     (visible_elements FFFEFF7F)
@@
     (tags "capacitor 0603")
     (attr smd)
-    (fp_text reference C1 (at -2.921 0 90) (layer F.SilkS)
+    (fp_text reference C1 (at 2.921 0 90) (layer F.SilkS)
       (effects (font (size 1 1) (thickness 0.15)))
     )
@@
     (pad "" thru_hole circle (at 5.08 -5.08 90) (size 3 3) (drill 2.05) (layers *.Cu *.Mask))
     (pad "" thru_hole circle (at -5.08 -5.08 90) (size 3 3) (drill 2.05) (layers *.Cu *.Mask))
+  )
+  (module lib_fp:LG_MARK_025in (layer B.Cu)
+    (at 93.091 140.335 270)
+    (fp_text reference G*** (at 0 0 270) (layer B.SilkS) hide
+      (effects (font (thickness 0.3)) (justify mirror))
+    )
+    (fp_text value LOGO (at 0.75 0 270) (layer B.SilkS) hide
+      (effects (font (thickness 0.3)) (justify mirror))
+    )
+    (fp_poly (pts (xy 3.132346 -0.010584) (xy 3.115552 -0.26543) (xy 3.070229 -0.56062) (xy 3.002782 -0.859373)
+      (xy 2.957264 -1.016) (xy 2.771313 -1.462202) (xy 2.513648 -1.874965) (xy 2.193538 -2.245544)
+      (xy 1.820254 -2.565194) (xy 1.403068 -2.825168) (xy 0.95125 -3.016723) (xy 0.783166 -3.066913)
+      (xy 0.619884 -3.099141) (xy 0.404805 -3.126273) (xy 0.164694 -3.146546) (xy -0.073682 -3.158202)
+      (xy -0.283555 -3.159479) (xy -0.438158 -3.148619) (xy -0.4445 -3.147639) (xy -0.938102 -3.029327)
+      (xy -1.405403 -2.840911) (xy -1.8346 -2.589255) (xy -2.213886 -2.281224) (xy -2.517635 -1.94209)
+      (xy -2.795012 -1.506941) (xy -2.99283 -1.043573) (xy -2.286001 -1.043573) (xy -2.255161 -1.180014)
+      (xy -2.16896 -1.356119) (xy -2.036873 -1.557108) (xy -1.868376 -1.768195) (xy -1.717261 -1.930855)
+      (xy -1.366873 -2.226972) (xy -0.98211 -2.448244) (xy -0.570448 -2.592574) (xy -0.139363 -2.657867)
+      (xy 0.303669 -2.642025) (xy 0.609768 -2.583373) (xy 0.813547 -2.521337) (xy 1.027916 -2.440572)
+      (xy 1.198623 -2.36241) (xy 1.431699 -2.212658) (xy 1.672697 -2.01088) (xy 1.899125 -1.779617)
+      (xy 2.088493 -1.541415) (xy 2.198706 -1.359984) (xy 2.283804 -1.16143) (xy 2.309716 -1.0143)
+      (xy 2.276453 -0.909483) (xy 2.199234 -0.845544) (xy 2.095652 -0.816628) (xy 1.999891 -0.852378)
+      (xy 1.902834 -0.95908) (xy 1.810907 -1.11327) (xy 1.594076 -1.436181) (xy 1.316605 -1.713238)
+      (xy 0.992292 -1.936052) (xy 0.634935 -2.096234) (xy 0.258331 -2.185397) (xy 0.021166 -2.201334)
+      (xy -0.366478 -2.160314) (xy -0.740465 -2.042505) (xy -1.087822 -1.855781) (xy -1.395578 -1.608017)
+      (xy -1.650761 -1.307086) (xy -1.767244 -1.115683) (xy -1.869519 -0.948452) (xy -1.960133 -0.851573)
+      (xy -1.999128 -0.831927) (xy -2.121347 -0.837118) (xy -2.225187 -0.902501) (xy -2.282249 -1.007123)
+      (xy -2.286001 -1.043573) (xy -2.99283 -1.043573) (xy -2.996925 -1.033982) (xy -3.089936 -0.657576)
+      (xy -1.211727 -0.657576) (xy -1.208474 -0.739205) (xy -1.181093 -0.815167) (xy -1.07134 -1.001006)
+      (xy -0.904972 -1.188621) (xy -0.706608 -1.355921) (xy -0.500867 -1.480814) (xy -0.390989 -1.524182)
+      (xy -0.22352 -1.553247) (xy -0.0103 -1.561287) (xy 0.212679 -1.549346) (xy 0.409428 -1.518469)
+      (xy 0.479046 -1.498938) (xy 0.675448 -1.400638) (xy 0.876944 -1.247505) (xy 1.056772 -1.06315)
+      (xy 1.186051 -0.875203) (xy 1.24348 -0.760531) (xy 1.262322 -0.688651) (xy 1.245429 -0.628523)
+      (xy 1.21351 -0.576258) (xy 1.111374 -0.481907) (xy 0.992447 -0.46149) (xy 0.879069 -0.513858)
+      (xy 0.812947 -0.596836) (xy 0.656714 -0.829517) (xy 0.48049 -0.985778) (xy 0.27185 -1.073524)
+      (xy 0.021166 -1.100667) (xy -0.248776 -1.064682) (xy -0.475172 -0.956248) (xy -0.659462 -0.774642)
+      (xy -0.677154 -0.750267) (xy -0.777913 -0.609654) (xy -0.847018 -0.525031) (xy -0.900272 -0.482272)
+      (xy -0.953477 -0.467249) (xy -0.995527 -0.465667) (xy -1.10493 -0.50453) (xy -1.168224 -0.57175)
+      (xy -1.211727 -0.657576) (xy -3.089936 -0.657576) (xy -3.122654 -0.525171) (xy -3.16252 -0.185718)
+      (xy -3.187575 0.169333) (xy -1.900705 0.168809) (xy -0.613834 0.168285) (xy -0.519073 0.021983)
+      (xy -0.368753 -0.140632) (xy -0.182518 -0.236763) (xy 0.023103 -0.266398) (xy 0.231584 -0.229524)
+      (xy 0.426397 -0.126127) (xy 0.574336 0.021122) (xy 0.687382 0.169333) (xy 3.132666 0.169333)
+      (xy 3.132346 -0.010584)) (layer B.SilkS) (width 0.01))
+    (fp_poly (pts (xy 0.51744 3.059553) (xy 1.016094 2.92595) (xy 1.01672 2.925729) (xy 1.357207 2.786503)
+      (xy 1.653321 2.620228) (xy 1.932547 2.409259) (xy 2.179379 2.17938) (xy 2.433745 1.9041)
+      (xy 2.629833 1.638516) (xy 2.785284 1.354849) (xy 2.917744 1.02532) (xy 2.924274 1.006579)
+      (xy 3.045624 0.656166) (xy 0.211666 0.633874) (xy 0.211666 0.47357) (xy 0.198985 0.355211)
+      (xy 0.167777 0.270865) (xy 0.160866 0.262466) (xy 0.065557 0.216031) (xy -0.041957 0.225713)
+      (xy -0.121859 0.287192) (xy -0.125511 0.29355) (xy -0.157817 0.396236) (xy -0.169334 0.505217)
+      (xy -0.169334 0.635) (xy -3.096039 0.635) (xy -3.066632 0.73025) (xy -2.936277 1.109492)
+      (xy -2.794156 1.427269) (xy -2.626804 1.706767) (xy -2.42076 1.971172) (xy -2.2225 2.183889)
+      (xy -1.83213 2.521198) (xy -1.405568 2.784178) (xy -0.950073 2.971165) (xy -0.472901 3.080498)
+      (xy 0.018689 3.110515) (xy 0.51744 3.059553)) (layer B.SilkS) (width 0.01))
+  )
+  (gr_text Out (at 110.236 131.2545) (layer B.SilkS)
+    (effects (font (size 1 1) (thickness 0.25)) (justify mirror))
+  )
+  (gr_text "Cg. Amp" (at 108.3945 137.795) (layer B.SilkS)
+    (effects (font (size 1 1) (thickness 0.25)) (justify mirror))
+  )
+  (gr_text Batt (at 110.0455 144.399) (layer B.SilkS)
+    (effects (font (size 1 1) (thickness 0.25)) (justify mirror))
+  )
+  (gr_text GND (at 109.982 147.0025) (layer B.SilkS)
+    (effects (font (size 1 1) (thickness 0.25)) (justify mirror))
+  )
+  (gr_text GND (at 109.982 140.335) (layer B.SilkS)
+    (effects (font (size 1 1) (thickness 0.25)) (justify mirror))
+  )
+  (gr_text GND (at 109.982 133.731) (layer B.SilkS)
+    (effects (font (size 1 1) (thickness 0.25)) (justify mirror))
+  )
+  (gr_text "Charge Amplifier\nLeeman Geophysical LLC\nRev.A - November 2017" (at 98.8695 140.7795 90) (layer B.SilkS)
+    (effects (font (size 1 1) (thickness 0.25)) (justify mirror))
   )
   (target plus (at 78.74 129.032) (size 5) (width 0.15) (layer Edge.Cuts))
@@
       )
     )
+  )
+  (zone (net 2) (net_name GNDA) (layer B.Cu) (hatch edge 0.508)
+    (connect_pads (clearance 0.1524))
+    (min_thickness 0.1524)
+    (fill yes (arc_segments 16) (thermal_gap 0.508) (thermal_bridge_width 0.508))
+    (polygon
+      (pts
+        (xy 115.062 152.146) (xy 78.994 152.146) (xy 79.0575 129.3495) (xy 115.062 129.286)
+      )
+    )
